Commit message: configured simulation environment

File: butlerbot_description/urdf/butlerbot_hokuyo.xacro (robot description, xacro)
@@ -2,5 +2,5 @@
 <robot name="hokuyo" xmlns:xacro="http://ros.org/wiki/xacro">
     <xacro:macro name="butlerbot_hokuyo" params="parent x_hok y_hok z_hok robot_name">
-        <link name="laser_sensor_link">
+        <link name="lidar_link">
             <inertial>
                 <mass value="1e-5" />
@@ -22,18 +22,18 @@
             </visual>
         </link>
-        <joint name="laser_sensor_joint" type="fixed">
+        <joint name="laser_joint" type="fixed">
             <origin xyz="${x_hok} ${y_hok} ${z_hok}" rpy="0 0 0" />
             <parent link="${parent}" />
-            <child link="laser_sensor_link" />
+            <child link="lidar_link" />
         </joint>
-        <gazebo reference="laser_sensor_link">
+        <gazebo reference="lidar_link">
             <sensor name="lidar" type="ray">
                 <always_on>true</always_on>
-                <visualize>false</visualize>
-                <update_rate>20</update_rate>
+                <visualize>true</visualize>
+                <update_rate>5</update_rate>
                 <ray>
                     <scan>
                         <horizontal>
-                            <samples>128</samples>
+                            <samples>360</samples>
                             <resolution>1.000000</resolution>
                             <min_angle>0.000000</min_angle>
@@ -58,5 +58,5 @@
                     </ros>
                     <output_type>sensor_msgs/LaserScan</output_type>
-                    <frame_name>${robot_name}/laser_sensor_link</frame_name>
+                    <frame_name>${robot_name}/laser_link</frame_name>
                 </plugin>
             </sensor>

File: butlerbot_description/urdf/butlerbot_kobuki.xacro (robot description, xacro)
@@ -130,19 +130,24 @@
         </joint>
         <!-- Kobuki's sensors -->
-        <!-- Gyroscope Sensor -->
-        <link name="gyro_link">
-            <inertial>
-                <mass value="0.001" />
-                <origin xyz="0 0 0" rpy="0 0 0" />
-                <inertia ixx="0.0001" ixy="0" ixz="0"
-                    iyy="0.000001" iyz="0"
-                    izz="0.0001" />
-            </inertial>
-        </link>
-        <joint name="gyro_joint" type="fixed">
-            <axis xyz="0 1 0" />
-            <origin xyz="0.056 0.062 0.0202" rpy="0 0 0" />
-            <parent link="base_link" />
-            <child link="gyro_link" />
+        <!-- IMU Sensor -->
+        <link name="imu_link">
+            <visual>
+                <geometry>
+                    <box size="0.05 0.05 0.05" />
+                </geometry>
+                <material name="red">
+                    <color rgba="1.0 0.2 0.2 1.0" />
+                </material>
+            </visual>
+            <collision>
+                <geometry>
+                    <box size="0.1 0.1 0.1" />
+                </geometry>
+            </collision>
+        </link>
+        <joint name="imu_joint" type="fixed">
+            <parent link="base_link" />
+            <child link="imu_link" />
+            <origin xyz="0 0 0.05" />
         </joint>
         <!-- Left Cliff Sensor -->

File: butlerbot_description/urdf/butlerbot_kobuki_gazebo.xacro (robot description, xacro)
@@ -113,9 +113,12 @@
 			</sensor>
 		</gazebo>
-		<gazebo reference="gyro_link">
-			<sensor type="imu" name="imu">
+		<gazebo reference="imu_link">
+			<sensor name="imu_sensor" type="imu">
+				<plugin filename="libgazebo_ros_imu_sensor.so" name="imu_plugin">
+					<initial_orientation_as_reference>false</initial_orientation_as_reference>
+				</plugin>
 				<always_on>true</always_on>
-				<update_rate>50</update_rate>
-				<visualize>false</visualize>
+				<update_rate>100</update_rate>
+				<visualize>true</visualize>
 				<imu>
 					<noise>
