Commit message: solved urdf issues

File: butlerbot_description/urdf/butlerbot.xacro (robot description, xacro)
@@ -1,6 +1,4 @@
 <?xml version="1.0"?>
 <robot xmlns:xacro="http://www.ros.org/wiki/xacro" name="butlerbot">
-    <xacro:arg name="robot_name" default="butlerbot_X" />
-    <xacro:property name="robot_name_prop" value="$(arg robot_name)" />
     <xacro:include filename="$(find butlerbot_description)/urdf/common_properties.xacro"/>
     <xacro:include filename="$(find butlerbot_description)/urdf/butlerbot_properties.xacro"/>
@@ -9,11 +7,6 @@
     <xacro:include filename="$(find butlerbot_description)/urdf/butlerbot_mod.xacro" />
     <xacro:include filename="$(find butlerbot_description)/urdf/butlerbot_hokuyo.xacro" />
-    <xacro:butlerbot_kobuki robot_name="$(arg robot_name)" />
-        <xacro:if value="${'butlerbot' in robot_name_prop}">
-            <xacro:butlerbot_mod bottom_parent="base_link" top_parent="base_link" />
-        </xacro:if>
-        <xacro:if value="${'mule' in robot_name_prop}">
-            <xacro:butlerbot_mod_mule bottom_parent="base_link" top_parent="base_link" />
-        </xacro:if>
-    <xacro:butlerbot_hokuyo parent="base_link" x_hok="0.103007" y_hok="0.0" z_hok="0.17" robot_name="$(arg robot_name)" />
+    <xacro:butlerbot_mod bottom_parent="base_link" top_parent="base_link" />
+    <xacro:butlerbot_mod_mule bottom_parent="base_link" top_parent="base_link" />
+    <xacro:butlerbot_hokuyo parent="base_link" x_hok="0.103007" y_hok="0.0" z_hok="0.17" />
 </robot>

File: butlerbot_description/urdf/butlerbot_hokuyo.xacro (robot description, xacro)
@@ -1,5 +1,5 @@
 <?xml version="1.0"?>
 <robot name="hokuyo" xmlns:xacro="http://ros.org/wiki/xacro">
-    <xacro:macro name="butlerbot_hokuyo" params="parent x_hok y_hok z_hok robot_name">
+    <xacro:macro name="butlerbot_hokuyo" params="parent x_hok y_hok z_hok">
         <link name="lidar_link">
             <inertial>
@@ -54,9 +54,8 @@
                 <plugin name="scan" filename="libgazebo_ros_ray_sensor.so">
                     <ros>
-                        <namespace>${robot_name}</namespace>
                         <remapping>~/out:=scan</remapping>
                     </ros>
                     <output_type>sensor_msgs/LaserScan</output_type>
-                    <frame_name>${robot_name}/laser_link</frame_name>
+                    <frame_name>lidar_link</frame_name>
                 </plugin>
             </sensor>

File: butlerbot_description/urdf/butlerbot_kobuki.xacro (robot description, xacro)
@@ -1,201 +1,197 @@
 <?xml version="1.0"?>
 <robot name="butlerbot_kobuki" xmlns:xacro="http://ros.org/wiki/xacro">
-    <xacro:arg name="robot_name" default="butlerbot_X" />
     <xacro:include filename="$(find butlerbot_description)/urdf/common_properties.xacro" />
     <xacro:include filename="$(find butlerbot_description)/urdf/butlerbot_kobuki_gazebo.xacro" />
-    <!-- Kobuki -->
-    <xacro:macro name="butlerbot_kobuki" params="robot_name">
-        <!-- Base Footprint -->
-        <link name="base_footprint" />
-        <!-- Base Link -->
-        <link name="base_link">
-            <visual>
-                <geometry>
-                    <mesh filename="package://butlerbot_description/meshes/kobuki/main_body.dae" />
-                </geometry>
-                <origin xyz="0.001 0 0.05199" rpy="0 0 0" />
-            </visual>
-            <collision>
-                <geometry>
-                    <cylinder length="0.10938" radius="0.178" />
-                </geometry>
-                <origin xyz="0.0 0 0.05949" rpy="0 0 0" />
-            </collision>
-            <inertial>
-                <origin xyz="0.01 0 0" />
-                <mass value="2.4" />
-                <inertia ixx="0.019995" ixy="0.0" ixz="0.0"
-                    iyy="0.019995" iyz="0.0"
-                    izz="0.03675" />
-            </inertial>
-        </link>
-        <joint name="base_joint" type="fixed">
-            <origin xyz="0 0 0.0102" rpy="0 0 0" />
-            <parent link="base_footprint" />
-            <child link="base_link" />
-        </joint>
-        <!-- Left Wheel -->
-        <link name="${robot_name}/wheel_left_link">
-            <visual>
-                <geometry>
-                    <mesh filename="package://butlerbot_description/meshes/wheel.dae" />
-                </geometry>
-                <origin rpy="0 0 0" xyz="0 0 0" />
-            </visual>
-            <collision>
-                <geometry>
-                    <cylinder length="0.0206" radius="0.0352" />
-                </geometry>
-                <origin rpy="0 0 0" xyz="0 0 0" />
-            </collision>
-            <inertial>
-                <mass value="0.01" />
-                <origin xyz="0 0 0" />
-                <inertia ixx="0.001" ixy="0.0" ixz="0.0" iyy="0.001" iyz="0.0" izz="0.001" />
-            </inertial>
-        </link>
-        <joint name="${robot_name}/joint_tire_left" type="continuous">
-            <parent link="base_link" />
-            <child link="${robot_name}/wheel_left_link" />
-            <origin rpy="-1.5707963267948966 0 0" xyz="0.00 0.115 0.0250" />
-            <axis xyz="0 0 1" />
-        </joint>
-        <!-- Right Wheel -->
-        <link name="${robot_name}/wheel_right_link">
-            <visual>
-                <geometry>
-                    <mesh filename="package://butlerbot_description/meshes/wheel.dae" />
-                </geometry>
-                <origin rpy="0 0 0" xyz="0 0 0" />
-            </visual>
-            <collision>
-                <geometry>
-                    <cylinder length="0.0206" radius="0.0350" />
-                </geometry>
-                <origin rpy="0 0 0" xyz="0 0 0" />
-            </collision>
-            <inertial>
-                <mass value="0.01" />
-                <origin xyz="0 0 0" />
-                <inertia ixx="0.001" ixy="0.0" ixz="0.0" iyy="0.001" iyz="0.0" izz="0.001" />
-            </inertial>
-        </link>
-        <joint name="${robot_name}/joint_tire_right" type="continuous">
-            <parent link="base_link" />
-            <child link="${robot_name}/wheel_right_link" />
-            <origin rpy="-1.5707963267948966 0 0" xyz="0.00 -0.115 0.0250" />
-            <axis xyz="0 0 1" />
-        </joint>
-        <!-- Front Castor Wheel -->
-        <link name="caster_front_link">
-            <collision>
-                <geometry>
-                    <cylinder length="0.0176" radius="0.017" />
-                </geometry>
-                <origin rpy="0 0 0" xyz="0 0 0" />
-            </collision>
-            <inertial>
-                <mass value="0.01" />
-                <origin xyz="0 0 0" />
-                <inertia ixx="0.001" ixy="0.0" ixz="0.0"
-                    iyy="0.001" iyz="0.0"
-                    izz="0.001" />
-            </inertial>
-        </link>
-        <joint name="caster_front_joint" type="fixed">
-            <parent link="base_link" />
-            <child link="caster_front_link" />
-            <origin xyz="0.115 0.0 0.007" rpy="${-M_PI/2} 0 0" />
-        </joint>
-        <!-- Back Castor Wheel -->
-        <link name="caster_back_link">
-            <collision>
-                <geometry>
-                    <cylinder length="0.0176" radius="0.017" />
-                </geometry>
-                <origin rpy="0 0 0" xyz="0 0 0" />
-            </collision>
-            <inertial>
-                <mass value="0.01" />
-                <origin xyz="0 0 0" />
-                <inertia ixx="0.001" ixy="0.0" ixz="0.0"
-                    iyy="0.001" iyz="0.0"
-                    izz="0.001" />
-            </inertial>
-        </link>
-        <joint name="caster_back_joint" type="fixed">
-            <parent link="base_link" />
-            <child link="caster_back_link" />
-            <origin xyz="-0.135 0.0 0.009" rpy="${-M_PI/2} 0 0" />
-        </joint>
-        <!-- Kobuki's sensors -->
-        <!-- IMU Sensor -->
-        <link name="imu_link">
-            <visual>
-                <geometry>
-                    <box size="0.05 0.05 0.05" />
-                </geometry>
-                <material name="red">
-                    <color rgba="1.0 0.2 0.2 1.0" />
-                </material>
-            </visual>
-            <collision>
-                <geometry>
-                    <box size="0.1 0.1 0.1" />
-                </geometry>
-            </collision>
-        </link>
-        <joint name="imu_joint" type="fixed">
-            <parent link="base_link" />
-            <child link="imu_link" />
-            <origin xyz="0 0 0.05" />
-        </joint>
-        <!-- Left Cliff Sensor -->
-        <link name="cliff_sensor_left_link">
-            <inertial>
-                <mass value="0.0001" />
-                <origin xyz="0 0 0" />
-                <inertia ixx="0.0001" ixy="0.0" ixz="0.0"
-                    iyy="0.0001" iyz="0.0"
-                    izz="0.0001" />
-            </inertial>
-        </link>
-        <joint name="cliff_sensor_left_joint" type="fixed">
-            <origin xyz="0.08734 0.13601 0.0214" rpy="0 ${M_PI/2} 0" />
-            <parent link="base_link" />
-            <child link="cliff_sensor_left_link" />
-        </joint>
-        <!-- Right Cliff Sensor -->
-        <link name="cliff_sensor_right_link">
-            <inertial>
-                <mass value="0.0001" />
-                <origin xyz="0 0 0" />
-                <inertia ixx="0.0001" ixy="0.0" ixz="0.0"
-                    iyy="0.0001" iyz="0.0"
-                    izz="0.0001" />
-            </inertial>
-        </link>
-        <joint name="cliff_sensor_right_joint" type="fixed">
-            <origin xyz="0.085 -0.13601 0.0214" rpy="0 ${M_PI/2} 0" />
-            <parent link="base_link" />
-            <child link="cliff_sensor_right_link" />
-        </joint>
-        <!-- Front Cliff Sensor -->
-        <link name="cliff_sensor_front_link">
-            <inertial>
-                <mass value="0.0001" />
-                <origin xyz="0 0 0" />
-                <inertia ixx="0.0001" ixy="0.0" ixz="0.0"
-                    iyy="0.0001" iyz="0.0"
-                    izz="0.0001" />
-            </inertial>
-        </link>
-        <joint name="cliff_sensor_front_joint" type="fixed">
-            <origin xyz="0.156 0.00 0.0214" rpy="0 ${M_PI/2} 0" />
-            <parent link="base_link" />
-            <child link="cliff_sensor_front_link" />
-        </joint>
-        <!-- Kobuki Gazebo simulation details -->
-        <xacro:kobuki_sim robot_name="$(arg robot_name)" />
-    </xacro:macro>
+    <!-- Base Link -->
+    <link name="base_link">
+        <visual>
+            <geometry>
+                <mesh filename="package://butlerbot_description/meshes/kobuki/main_body.dae" />
+            </geometry>
+            <origin xyz="0.001 0 0.05199" rpy="0 0 0" />
+        </visual>
+        <collision>
+            <geometry>
+                <cylinder length="0.10938" radius="0.178" />
+            </geometry>
+            <origin xyz="0.0 0 0.05949" rpy="0 0 0" />
+        </collision>
+        <inertial>
+            <origin xyz="0.01 0 0" />
+            <mass value="2.4" />
+            <inertia ixx="0.019995" ixy="0.0" ixz="0.0"
+                iyy="0.019995" iyz="0.0"
+                izz="0.03675" />
+        </inertial>
+    </link>
+    <!-- Base Footprint -->
+    <link name="base_footprint" />
+    <joint name="base_joint" type="fixed">
+        <origin xyz="0 0 0.0102" rpy="0 0 0" />
+        <parent link="base_link" />
+        <child link="base_footprint" />
+    </joint>
+    <!-- Left Wheel -->
+    <link name="wheel_left_link">
+        <visual>
+            <geometry>
+                <mesh filename="package://butlerbot_description/meshes/wheel.dae" />
+            </geometry>
+            <origin rpy="0 0 0" xyz="0 0 0" />
+        </visual>
+        <collision>
+            <geometry>
+                <cylinder length="0.0206" radius="0.0352" />
+            </geometry>
+            <origin rpy="0 0 0" xyz="0 0 0" />
+        </collision>
+        <inertial>
+            <mass value="0.01" />
+            <origin xyz="0 0 0" />
+            <inertia ixx="0.001" ixy="0.0" ixz="0.0" iyy="0.001" iyz="0.0" izz="0.001" />
+        </inertial>
+    </link>
+    <joint name="joint_tire_left" type="continuous">
+        <parent link="base_link" />
+        <child link="wheel_left_link" />
+        <origin rpy="-1.5707963267948966 0 0" xyz="0.00 0.115 0.0250" />
+        <axis xyz="0 0 1" />
+    </joint>
+    <!-- Right Wheel -->
+    <link name="wheel_right_link">
+        <visual>
+            <geometry>
+                <mesh filename="package://butlerbot_description/meshes/wheel.dae" />
+            </geometry>
+            <origin rpy="0 0 0" xyz="0 0 0" />
+        </visual>
+        <collision>
+            <geometry>
+                <cylinder length="0.0206" radius="0.0350" />
+            </geometry>
+            <origin rpy="0 0 0" xyz="0 0 0" />
+        </collision>
+        <inertial>
+            <mass value="0.01" />
+            <origin xyz="0 0 0" />
+            <inertia ixx="0.001" ixy="0.0" ixz="0.0" iyy="0.001" iyz="0.0" izz="0.001" />
+        </inertial>
+    </link>
+    <joint name="joint_tire_right" type="continuous">
+        <parent link="base_link" />
+        <child link="wheel_right_link" />
+        <origin rpy="-1.5707963267948966 0 0" xyz="0.00 -0.115 0.0250" />
+        <axis xyz="0 0 1" />
+    </joint>
+    <!-- Front Castor Wheel -->
+    <link name="caster_front_link">
+        <collision>
+            <geometry>
+                <cylinder length="0.0176" radius="0.017" />
+            </geometry>
+            <origin rpy="0 0 0" xyz="0 0 0" />
+        </collision>
+        <inertial>
+            <mass value="0.01" />
+            <origin xyz="0 0 0" />
+            <inertia ixx="0.001" ixy="0.0" ixz="0.0"
+                iyy="0.001" iyz="0.0"
+                izz="0.001" />
+        </inertial>
+    </link>
+    <joint name="caster_front_joint" type="fixed">
+        <parent link="base_link" />
+        <child link="caster_front_link" />
+        <origin xyz="0.115 0.0 0.007" rpy="${-M_PI/2} 0 0" />
+    </joint>
+    <!-- Back Castor Wheel -->
+    <link name="caster_back_link">
+        <collision>
+            <geometry>
+                <cylinder length="0.0176" radius="0.017" />
+            </geometry>
+            <origin rpy="0 0 0" xyz="0 0 0" />
+        </collision>
+        <inertial>
+            <mass value="0.01" />
+            <origin xyz="0 0 0" />
+            <inertia ixx="0.001" ixy="0.0" ixz="0.0"
+                iyy="0.001" iyz="0.0"
+                izz="0.001" />
+        </inertial>
+    </link>
+    <joint name="caster_back_joint" type="fixed">
+        <parent link="base_link" />
+        <child link="caster_back_link" />
+        <origin xyz="-0.135 0.0 0.009" rpy="${-M_PI/2} 0 0" />
+    </joint>
+    <!-- Kobuki's sensors -->
+    <!-- IMU Sensor -->
+    <link name="imu_link">
+        <visual>
+            <geometry>
+                <box size="0.05 0.05 0.05" />
+            </geometry>
+            <material name="red">
+                <color rgba="1.0 0.2 0.2 1.0" />
+            </material>
+        </visual>
+        <collision>
+            <geometry>
+                <box size="0.1 0.1 0.1" />
+            </geometry>
+        </collision>
+    </link>
+    <joint name="imu_joint" type="fixed">
+        <parent link="base_link" />
+        <child link="imu_link" />
+        <origin xyz="0 0 0.05" />
+    </joint>
+    <!-- Left Cliff Sensor -->
+    <link name="cliff_sensor_left_link">
+        <inertial>
+            <mass value="0.0001" />
+            <origin xyz="0 0 0" />
+            <inertia ixx="0.0001" ixy="0.0" ixz="0.0"
+                iyy="0.0001" iyz="0.0"
+                izz="0.0001" />
+        </inertial>
+    </link>
+    <joint name="cliff_sensor_left_joint" type="fixed">
+        <origin xyz="0.08734 0.13601 0.0214" rpy="0 ${M_PI/2} 0" />
+        <parent link="base_link" />
+        <child link="cliff_sensor_left_link" />
+    </joint>
+    <!-- Right Cliff Sensor -->
+    <link name="cliff_sensor_right_link">
+        <inertial>
+            <mass value="0.0001" />
+            <origin xyz="0 0 0" />
+            <inertia ixx="0.0001" ixy="0.0" ixz="0.0"
+                iyy="0.0001" iyz="0.0"
+                izz="0.0001" />
+        </inertial>
+    </link>
+    <joint name="cliff_sensor_right_joint" type="fixed">
+        <origin xyz="0.085 -0.13601 0.0214" rpy="0 ${M_PI/2} 0" />
+        <parent link="base_link" />
+        <child link="cliff_sensor_right_link" />
+    </joint>
+    <!-- Front Cliff Sensor -->
+    <link name="cliff_sensor_front_link">
+        <inertial>
+            <mass value="0.0001" />
+            <origin xyz="0 0 0" />
+            <inertia ixx="0.0001" ixy="0.0" ixz="0.0"
+                iyy="0.0001" iyz="0.0"
+                izz="0.0001" />
+        </inertial>
+    </link>
+    <joint name="cliff_sensor_front_joint" type="fixed">
+        <origin xyz="0.156 0.00 0.0214" rpy="0 ${M_PI/2} 0" />
+        <parent link="base_link" />
+        <child link="cliff_sensor_front_link" />
+    </joint>
+    <!-- Kobuki Gazebo simulation details -->
+    <xacro:kobuki_sim />
 </robot>

File: butlerbot_description/urdf/butlerbot_kobuki_gazebo.xacro (robot description, xacro)
@@ -1,6 +1,5 @@
 <?xml version="1.0"?>
 <robot name="kobuki_sim" xmlns:xacro="http://ros.org/wiki/xacro">
-	<xacro:arg name="robot_name" default="butlerbot_X" />
-	<xacro:macro name="kobuki_sim" params="robot_name">
+	<xacro:macro name="kobuki_sim" >
 		<gazebo reference="wheel_left_link">
 			<mu1>1.0</mu1>
@@ -118,4 +117,7 @@
 					<initial_orientation_as_reference>false</initial_orientation_as_reference>
 				</plugin>
+				<ros>
+					<remapping>~/out:=imu</remapping>
+				</ros>
 				<always_on>true</always_on>
 				<update_rate>100</update_rate>
@@ -142,12 +144,7 @@
 		<gazebo>
 			<plugin name='diff_drive' filename='libgazebo_ros_diff_drive.so'>
-				<ros>
-					<namespace>/</namespace>
-					<argument>cmd_vel:=${robot_name}/cmd_vel</argument>
-					<argument>odom:=${robot_name}/odom</argument>
-				</ros>
 				<!-- wheels -->
-				<left_joint>${robot_name}/joint_tire_left</left_joint>
-				<right_joint>${robot_name}/joint_tire_right</right_joint>
+				<left_joint>oint_tire_left</left_joint>
+				<right_joint>joint_tire_right</right_joint>
 				<!-- kinematics -->
 				<wheel_separation>0.4</wheel_separation>
@@ -160,6 +157,6 @@
 				<publish_odom_tf>true</publish_odom_tf>
 				<publish_wheel_tf>true</publish_wheel_tf>
-				<odometry_frame>${robot_name}/odom</odometry_frame>
-				<robot_base_frame>${robot_name}/base_footprint</robot_base_frame>
+				<odometry_frame>odom</odometry_frame>
+				<robot_base_frame>base_footprint</robot_base_frame>
 			</plugin>
 		</gazebo>

File: butlerbot_description/urdf/butlerbot_mod.xacro (robot description, xacro)
@@ -10,16 +10,5 @@
                 <origin xyz="0 0 0" rpy="0 0 0" />
                 <geometry>
-                    <xacro:if value="${robot_name_prop == 'butlerbot_1'}">
-                        <mesh
-                            filename="package://butlerbot_description/meshes/butlerbot/TOP_colour_1.dae" />
-                    </xacro:if>
-                    <xacro:if value="${robot_name_prop == 'butlerbot_2'}">
-                        <mesh
-                            filename="package://butlerbot_description/meshes/butlerbot/TOP_colour_2.dae" />
-                    </xacro:if>
-                    <xacro:if
-                        value="${robot_name_prop != 'butlerbot_1' and robot_name_prop != 'butlerbot_2'}">
-                        <mesh filename="package://butlerbot_description/meshes/butlerbot/TOP_colour.dae" />
-                    </xacro:if>
+                        <mesh filename="package://butlerbot_description/meshes/butlerbot/TOP_colour_1.dae" />
                 </geometry>
             </visual>
@@ -48,17 +37,5 @@
                 <origin xyz="0 0 0" rpy="0 0 0" />
                 <geometry>
-                    <xacro:if value="${robot_name_prop == 'butlerbot_1'}">
-                        <mesh
-                            filename="package://butlerbot_description/meshes/butlerbot/BOTTOM_colour_1.dae" />
-                    </xacro:if>
-                    <xacro:if value="${robot_name_prop == 'butlerbot_2'}">
-                        <mesh
-                            filename="package://butlerbot_description/meshes/butlerbot/BOTTOM_colour_2.dae" />
-                    </xacro:if>
-                    <xacro:if
-                        value="${robot_name_prop != 'butlerbot_1' and robot_name_prop != 'butlerbot_2'}">
-                        <mesh
-                            filename="package://butlerbot_description/meshes/butlerbot/BOTTOM_colour.dae" />
-                    </xacro:if>
+                        <mesh filename="package://butlerbot_description/meshes/butlerbot/BOTTOM_colour_1.dae" />
                 </geometry>
             </visual>
@@ -79,5 +56,5 @@
     <!-- Mule Related -->
     <xacro:macro name="butlerbot_mod_mule" params="bottom_parent top_parent">
-        <link name="butlerbot_top_link">
+        <link name="mule_butlerbot_top_link">
             <visual>
                 <origin xyz="0 0 0" rpy="0 0 0" />
@@ -101,10 +78,10 @@
             </inertial>
         </link>
-        <joint name="butlerbot_top_joint" type="fixed">
+        <joint name="mule_butlerbot_top_joint" type="fixed">
             <origin xyz="0.00364 0.0 0.24583" rpy="0 0 0" />
             <parent link="${top_parent}" />
-            <child link="butlerbot_top_link" />
+            <child link="mule_butlerbot_top_link" />
         </joint>
-        <link name="butlerbot_bottom_link">
+        <link name="mule_butlerbot_bottom_link">
             <visual>
                 <origin xyz="0 0 0" rpy="0 0 0" />
@@ -121,8 +98,8 @@
             </inertial>
         </link>
-        <joint name="butlerbot_bottom_joint" type="fixed">
+        <joint name="mule_butlerbot_bottom_joint" type="fixed">
             <origin xyz="0.001 0.0 0.12" rpy="0 0 0" />
             <parent link="${bottom_parent}" />
-            <child link="butlerbot_bottom_link" />
+            <child link="mule_butlerbot_bottom_link" />
         </joint>
     </xacro:macro>
